Commit message: Added robot description and Adjusted height of the robot

File: src/agri_robot_description/urdf/assembly_robot.urdf (robot description, URDF)
Before this commit: robot assembly_robot, 9 links, 8 joints
Links:
- link base_footprint: geometry 
Joints:
- joint base_footprint_joint: origin xyz=0 0 0.001 rpy=0 0 0 -> xyz=0 0 0.225 rpy=0 0 0

Commit message: [ADD]  - Lidar odometry pkg called RF2O  - Adjust the wheel frames to be shown in rviz  - Adjust the frames

File: src/agri_robot_description/urdf/assembly_robot.urdf (robot description, URDF)
Before this commit: robot assembly_robot, 9 links, 8 joints
Links:
- removed link base_footprint
Joints:
- removed joint base_footprint_joint
- joint Front_Left_Wheel_Joint: axis 1 0 0 -> 0 0 0; type continuous -> fixed
- joint Front_Right_Wheel_Joint: axis 1 0 0 -> 0 0 0; type continuous -> fixed
- joint Lidar_Joint: origin xyz=0.0815 -0.005 0.3095 rpy=0 0 0 -> xyz=0.0815 -0.005 0.3095 rpy=0 0 3.14
- joint Rear_Left_Wheel_Link: axis 1 0 0 -> 0 0 0; type continuous -> fixed
- joint Rear_Right_Wheel_Joint: axis 1 0 0 -> 0 0 0; type continuous -> fixed
